Commit message: world update

File: oparm_description/urdf/oparm.xacro (robot description, xacro)
@@ -6,4 +6,10 @@
 	<!-- END - Include -->
 	<!-- BGN - Robot description -->
+	  <!-- Used for fixing robot to Gazebo 'base_link' -->
+    <link name="world"/>
+    <joint name="fixed" type="fixed">
+        <parent link="world"/>
+        <child link="${l00}"/>
+    </joint>
 	<m_link_mesh name="${l00}"
 							 origin_rpy="0 0 0" origin_xyz="0 0 0"
